File: HARDWARE/EDA/KICAD/CDJC/CDJC.sch (KiCad schematic (older format))
At the start: 68 parts

Commit message: finished project
Parts:
- added U? (x14): 74LS32, symbol 74xx:74LS32
- added U? (x7): 74LS08, symbol 74xx:74LS08
- added U? (x6): 74LS04, symbol 74xx:74LS04
- J?: footprint Connector_PinHeader_2.00mm:PinHeader_1x03_P2.00mm_Horizontal -> Connector_PinSocket_2.00mm:PinSocket_1x03_P2.00mm_Horizontal
- J?: footprint Connector_PinHeader_2.00mm:PinHeader_1x05_P2.00mm_Horizontal -> Connector_PinSocket_2.00mm:PinSocket_1x05_P2.00mm_Horizontal
- J?: footprint Connector_PinHeader_2.00mm:PinHeader_1x08_P2.00mm_Horizontal -> Connector_PinSocket_2.00mm:PinSocket_1x08_P2.00mm_Horizontal
Connections:
- net +5VD: now also U?.14 (VCC), U?.14 (VCC), U?.14 (VCC), U?.14 (VCC), U?.14 (VCC), U?.14 (VCC)
- net EI: now also U?.4
- net ELMon: now also U?.4
- net FBMon: now also U?.10, U?.10, U?.13, U?.2
- net GNDD: now also U?.11, U?.12, U?.13, U?.13, U?.3, U?.5, U?.7 (GND), U?.7 (GND), U?.7 (GND), U?.7 (GND), U?.7 (GND), U?.7 (GND), U?.9
- net LBLBI: now also U?.12
- net LBMon: now also U?.10, U?.10, U?.2, U?.5
- net MRI: now also U?.9
- net MRLMon: now also U?.12
- net NBMon: now also U?.1, U?.1, U?.9, U?.9, U?.9
- net at U?.13 (CKEN): now also U?.3
- net at U?.15 (Reset): now also U?.6
- net at D?.1 (K), U?.3, U?.9: now also U?.13, U?.2
- net at U?.5: now also U?.8
- net at U?.1: now also U?.8
- new net: U?.10, U?.3
- new net: U?.1, U?.11
- new net: U?.12, U?.3
- new net: U?.13, U?.6
- new net: U?.11, U?.5
- new net: U?.1, U?.6
- new net: U?.2, U?.3
- new net: U?.11, U?.4
- new net: U?.5, U?.8
- new net: U?.12, U?.8
- new net: U?.11, U?.13
- no-connect marks 2 -> 8
Other:
- moved on the sheet: C?, D?, J?, R?, SW?, U?, U?A, U?B, U?C, U?D, U?E, U?G

Commit message: finished project
Parts:
- removed C? (x4): 100nF 63V, Capacitor_THT:C_Rect_L7.0mm_W2.5mm_P5.00mm, symbol Device:C
- removed U? (x8): 74LS32, symbol 74xx:74LS32
- removed U? (x4): 74LS08, symbol 74xx:74LS08
- removed U? (x7): 74LS04, symbol 74xx:74LS04
- added C? (x8): 100nF 63V, Capacitor_THT:C_Rect_L7.0mm_W2.5mm_P5.00mm, symbol Device:C
- added D? (x3): 1N4148, Diode_THT:D_DO-35_SOD27_P7.62mm_Horizontal, symbol Diode:1N4148
- added Q?: BC549, Package_TO_SOT_THT:TO-92_Inline, symbol Transistor_BJT:BC549
- added R? (x4): 300K, Resistor_THT:R_Axial_DIN0207_L6.3mm_D2.5mm_P7.62mm_Horizontal, symbol Device:R
- added R?: 1K, Resistor_THT:R_Axial_DIN0207_L6.3mm_D2.5mm_P7.62mm_Horizontal, symbol Device:R
- added R?: 150K, Resistor_THT:R_Axial_DIN0207_L6.3mm_D2.5mm_P7.62mm_Horizontal, symbol Device:R
- added U? (x4): 74LS08, Package_DIP:DIP-14_W7.62mm_LongPads, symbol 74xx:74LS08
- added U? (x4): 74LS32, Package_DIP:DIP-14_W7.62mm_LongPads, symbol 74xx:74LS32
- U? (x34): footprint (none) -> Package_DIP:DIP-14_W7.62mm_LongPads
Connections:
- net !LBO: now also D?.1 (K); no longer U?.6
- net +5VD: now also C?.1, C?.1, C?.1, C?.1, C?.1, C?.1, C?.1, C?.1, R?.2, U?.14 (VCC), U?.14 (VCC), U?.14 (VCC), U?.14 (VCC), U?.14 (VCC)
- net EI: now also U?.1, R?.1; no longer U?.4
- net FBMon: now also U?.10; no longer U?.13
- net FBO: now also D?.1 (K); no longer U?.3
- net GNDD: now also C?.2, C?.2, C?.2, C?.2, C?.2, C?.2, C?.2, C?.2, Q?.3 (E), R?.1, R?.2, R?.2, R?.2, U?.12, U?.12, U?.12, U?.13, U?.13, U?.13, U?.7 (GND), U?.7 (GND), U?.7 (GND), U?.7 (GND), U?.7 (GND)
- net LBLBI: now also U?.9, R?.1; no longer J?.3 (Pin_3), U?.12, U?.8
- net LBMon: now also U?.10, U?.13; no longer U?.10, U?.2
- net MRI: now also U?.5, R?.1; no longer U?.9
- net MRLMon: now also U?.1; no longer U?.12
- net NBMon: now also U?.9; no longer U?.1
- net at U?.3: now also U?.10, U?.10, U?.5; no longer U?.12
- net at U?.6: now also U?.9; no longer U?.13
- net at D?.1 (K): now also U?.4; no longer U?.2
- net at U?.5: now also U?.3; no longer U?.11
- net at U?.1: now also U?.3; no longer U?.6
- net at U?.2: now also U?.11; no longer U?.3
- net at U?.12: now also U?.6; no longer U?.8
- net at U?.13: now also U?.8; no longer U?.11
- net EB_SW renamed LB_SW
- new net: U?.2, U?.4, U?.8
- new net: U?.12, U?.8
- new net: D?.1 (K), R?.2, U?.12, U?.13, U?.2
- new net: D?.2 (A), U?.8
- new net: Q?.1 (C), R?.1, U?.9
- new net: D?.2 (A), U?.6
- new net: D?.2 (A), U?.11
- new net: Q?.2 (B), R?.1, R?.2
- new net LBLBO: D?.1 (K), J?.3 (Pin_3)
- no-connect marks 8 -> 4
Other:
- moved on the sheet: C?, D?, J?, U?, U?A, U?B, U?D, U?E

Commit message: paused PCB design
Parts:
- D10, D11, D13, D14, D15, D16, D17, D18, D19, D20, D21, D9: renamed from D?; footprint Diode_THT:D_DO-35_SOD27_P7.62mm_Horizontal -> Diode_THT:D_DO-34_SOD68_P2.54mm_Vertical_AnodeUp
- D12: renamed from D?; footprint Diode_THT:D_DO-35_SOD27_P7.62mm_Horizontal -> Diode_THT:D_DO-34_SOD68_P7.62mm_Horizontal
- R1, R10, R11, R12, R13, R14, R15, R16, R17, R2, R3, R4, R5, R6, R7, R8, R9: renamed from R?; footprint Resistor_THT:R_Axial_DIN0207_L6.3mm_D2.5mm_P7.62mm_Horizontal -> Resistor_THT:R_Axial_DIN0204_L3.6mm_D1.6mm_P5.08mm_Horizontal
- gave numbers to parts that had none: 34
Connections:
- net ELMon: now also U7.1; no longer U7.4
- net FBMon: now also U7.10; no longer U7.2
- net GNDD: now also U3.12, U3.13; no longer U4.12, U4.13
- net LBMon: now also U7.2; no longer U7.5
- net LB_SW: now also U4.13; no longer U3.13
- net MRI: now also U6.5; no longer U5.5
- net MRLMon: now also U4.11, U6.12; no longer U3.11, U5.1
- net NBMon: now also U7.9; no longer U7.1
- net at U4.8: now also U4.12; no longer U3.12
- net at U6.2, U8.8: now also U6.4; no longer U5.4
- net at U7.8: now also U5.10, U5.5, U7.5; no longer U6.12
- net at U7.6: now also U5.1; no longer U7.9
- net at D21.1 (K): now also U5.9; no longer U6.4
- net at U5.8: now also D20.2 (A); no longer D12.2 (A)
- net at Q1.1 (C), R17.1: now also U5.4; no longer U5.9
- net at U6.6: now also U8.12; no longer D20.2 (A)
- net at U5.3: now also U8.2; no longer U8.5
- net at U6.11: now also U8.5; no longer U8.2
- net at U5.6: now also D12.2 (A); no longer U8.12
- new net: U7.3, U7.4
Other:
- moved on the sheet: D10, D11, D12, D13, D14, D15, D16, D17, D18, D19, D20, D21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

Commit message: i am crazy
Parts:
- removed C1: 1800µF 6.3V, Capacitor_THT:CP_Radial_D10.0mm_P5.00mm, symbol Device:CP
Changed lines of the file:
@@
 	10100 2450 10100 2500
-$Comp
-L Device:CP C1
-U 1 1 6187897F
-P 6950 2650
-F 0 "C1" V 7050 2400 50  0000 L CNN
-F 1 "1800µF 6.3V" V 6750 2400 50  0000 L CNN
-F 2 "Capacitor_THT:CP_Radial_D10.0mm_P5.00mm" H 6988 2500 50  0001 C CNN
-F 3 "~" H 6950 2650 50  0001 C CNN
-	1    6950 2650
-	1    0    0    -1
-$EndComp
-$Comp
-L power:GNDD #PWR025
-U 1 1 61878FA8
-P 6950 2850
-F 0 "#PWR025" H 6950 2600 50  0001 C CNN
-F 1 "GNDD" H 6954 2695 50  0000 C CNN
-F 2 "" H 6950 2850 50  0001 C CNN
-F 3 "" H 6950 2850 50  0001 C CNN
-	1    6950 2850
-	1    0    0    -1
-$EndComp
-Wire Wire Line
-	6950 2850 6950 2800
-$Comp
-L power:+5VD #PWR024
-U 1 1 6187CA57
-P 6950 2450
-F 0 "#PWR024" H 6950 2300 50  0001 C CNN
-F 1 "+5VD" H 6965 2623 50  0000 C CNN
-F 2 "" H 6950 2450 50  0001 C CNN
-F 3 "" H 6950 2450 50  0001 C CNN
-	1    6950 2450
-	1    0    0    -1
-$EndComp
-Wire Wire Line
-	6950 2450 6950 2500
 $Comp
 L power:+5VD #PWR021
