File: HARDWARE/EDA/KICAD/CDJC/_autosave-CDJC.sch (KiCad schematic (older format))
At the start: 63 parts, among them J1 COM_IN, J2 COM_OUT, J3 POWER_IN, J4 POWER_OUT, J5 BIT_OUT, Q1 BC549, SW1 B-SET, U1 74LS04, U2 74LS32, U3 74LS08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

Commit message: i am crazy
Connections:
- net FB_SW: now also U2.12; no longer U2.4
- net GNDD: now also U2.1, U2.2; no longer U2.12, U2.13
- net LB_SW: now also U2.10; no longer U2.1
- net NB_SW: now also U2.13, U2.4; no longer U2.10, U2.2
- net at U2.6: now also U1.9; no longer U1.11
- net at U2.8: now also U1.11; no longer U1.13
- net at U2.3: no longer U1.9
- net at U2.11: now also U1.13
Other:
- moved on the sheet: U2A, U2B, U2C, U2D
Changed lines of the file:
@@
 Text Notes 2050 3900 2    50   ~ 0
 FB:1, NB:0, LB:0
+Text GLabel 1050 4100 0    50   Input ~ 0
+NB_SW
 Text GLabel 1050 4300 0    50   Input ~ 0
-NB_SW
-Text GLabel 1050 4100 0    50   Input ~ 0
 LB_SW
 Text GLabel 2300 4750 2    50   Output ~ 0
 FBMon
-$Comp
-L 74xx:74LS32 U2
-U 1 1 616AA084
-P 1500 4200
-F 0 "U2" H 1750 4100 50  0000 C CNN
-F 1 "74LS32" H 1750 4300 50  0000 C CNN
-F 2 "Package_DIP:DIP-14_W7.62mm_LongPads" H 1500 4200 50  0001 C CNN
-F 3 "http://www.ti.com/lit/gpn/sn74LS32" H 1500 4200 50  0001 C CNN
-	1    1500 4200
-	1    0    0    -1
-$EndComp
 Wire Wire Line
 	1050 4100 1200 4100
@@
 L 74xx:74LS32 U2
 U 2 1 615E6CA6
-P 1500 5550
-F 0 "U2" H 1750 5450 50  0000 C CNN
-F 1 "74LS32" H 1750 5650 50  0000 C CNN
-F 2 "Package_DIP:DIP-14_W7.62mm_LongPads" H 1500 5550 50  0001 C CNN
-F 3 "http://www.ti.com/lit/gpn/sn74LS32" H 1500 5550 50  0001 C CNN
-	2    1500 5550
+P 1500 4200
+F 0 "U2" H 1750 4100 50  0000 C CNN
+F 1 "74LS32" H 1750 4300 50  0000 C CNN
+F 2 "Package_DIP:DIP-14_W7.62mm_LongPads" H 1500 4200 50  0001 C CNN
+F 3 "http://www.ti.com/lit/gpn/sn74LS32" H 1500 4200 50  0001 C CNN
+	2    1500 4200
 	1    0    0    -1
 $EndComp
@@
 Text GLabel 2300 7450 2    50   Output ~ 0
 LBMon
-$Comp
-L 74xx:74LS32 U2
-U 3 1 6161ACD8
-P 1500 6900
-F 0 "U2" H 1750 6800 50  0000 C CNN
-F 1 "74LS32" H 1750 7000 50  0000 C CNN
-F 2 "Package_DIP:DIP-14_W7.62mm_LongPads" H 1500 6900 50  0001 C CNN
-F 3 "http://www.ti.com/lit/gpn/sn74LS32" H 1500 6900 50  0001 C CNN
-	3    1500 6900
-	1    0    0    -1
-$EndComp
 Wire Wire Line
 	1050 6800 1200 6800
@@
 L 74xx:74LS32 U2
 U 4 1 64C646E2
-P 10850 1350
-F 0 "U2" H 11100 1250 50  0000 C CNN
-F 1 "74LS32" H 10850 1550 50  0000 C CNN
-F 2 "Package_DIP:DIP-14_W7.62mm_LongPads" H 10850 1350 50  0001 C CNN
-F 3 "http://www.ti.com/lit/gpn/sn74LS32" H 10850 1350 50  0001 C CNN
-	4    10850 1350
+P 1500 6900
+F 0 "U2" H 1750 6800 50  0000 C CNN
+F 1 "74LS32" H 1500 7100 50  0000 C CNN
+F 2 "Package_DIP:DIP-14_W7.62mm_LongPads" H 1500 6900 50  0001 C CNN
+F 3 "http://www.ti.com/lit/gpn/sn74LS32" H 1500 6900 50  0001 C CNN
+	4    1500 6900
 	1    0    0    -1
 $EndComp
@@
 	1    0    0    -1
 $EndComp
+$Comp
+L 74xx:74LS32 U2
+U 3 1 6161ACD8
+P 1500 5550
+F 0 "U2" H 1750 5450 50  0000 C CNN
+F 1 "74LS32" H 1750 5650 50  0000 C CNN
+F 2 "Package_DIP:DIP-14_W7.62mm_LongPads" H 1500 5550 50  0001 C CNN
+F 3 "http://www.ti.com/lit/gpn/sn74LS32" H 1500 5550 50  0001 C CNN
+	3    1500 5550
+	1    0    0    -1
+$EndComp
+$Comp
+L 74xx:74LS32 U2
+U 1 1 616AA084
+P 10850 1350
+F 0 "U2" H 11100 1250 50  0000 C CNN
+F 1 "74LS32" H 11100 1450 50  0000 C CNN
+F 2 "Package_DIP:DIP-14_W7.62mm_LongPads" H 10850 1350 50  0001 C CNN
+F 3 "http://www.ti.com/lit/gpn/sn74LS32" H 10850 1350 50  0001 C CNN
+	1    10850 1350
+	1    0    0    -1
+$EndComp

Commit message: PCI connector OK
Connections:
- net at U2.6: now also U1.13; no longer U1.9
- net at U1.12: now also U3.1; no longer U3.9
- net at U2.11: now also U1.9; no longer U1.13
- net at U1.8: now also U3.9; no longer U3.1
Other:
- moved on the sheet: U1D, U1F
Changed lines of the file:
@@
 L 74xx:74LS04 U1
 U 6 1 6161ACE0
-P 2200 6900
-F 0 "U1" H 2450 6800 50  0000 C CNN
-F 1 "74LS04" H 2450 7000 50  0000 C CNN
-F 2 "Package_DIP:DIP-14_W7.62mm_LongPads" H 2200 6900 50  0001 C CNN
-F 3 "http://www.ti.com/lit/gpn/sn74LS04" H 2200 6900 50  0001 C CNN
-	6    2200 6900
+P 2200 4200
+F 0 "U1" H 2450 4100 50  0000 C CNN
+F 1 "74LS04" H 2450 4300 50  0000 C CNN
+F 2 "Package_DIP:DIP-14_W7.62mm_LongPads" H 2200 4200 50  0001 C CNN
+F 3 "http://www.ti.com/lit/gpn/sn74LS04" H 2200 4200 50  0001 C CNN
+	6    2200 4200
 	1    0    0    -1
 $EndComp
@@
 L 74xx:74LS04 U1
 U 4 1 616B3BFE
-P 2200 4200
-F 0 "U1" H 2450 4100 50  0000 C CNN
-F 1 "74LS04" H 2450 4300 50  0000 C CNN
-F 2 "Package_DIP:DIP-14_W7.62mm_LongPads" H 2200 4200 50  0001 C CNN
-F 3 "http://www.ti.com/lit/gpn/sn74LS04" H 2200 4200 50  0001 C CNN
-	4    2200 4200
+P 2200 6900
+F 0 "U1" H 2450 6800 50  0000 C CNN
+F 1 "74LS04" H 2450 7000 50  0000 C CNN
+F 2 "Package_DIP:DIP-14_W7.62mm_LongPads" H 2200 6900 50  0001 C CNN
+F 3 "http://www.ti.com/lit/gpn/sn74LS04" H 2200 6900 50  0001 C CNN
+	4    2200 6900
 	1    0    0    -1
 $EndComp
