File: HARDWARE/EDA/KICAD/CDJC/_autosave-CDJC.sch (KiCad schematic (older format))
At the start: 55 parts, among them J1 COM_IN, J2 COM_OUT, J3 POWER_IN, J4 POWER_OUT, J5 BIT_OUT, Q1 BC549, SW1 B-SET, U1 74LS04, U2 74LS32, U3 74LS08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

Commit message: i am crazy
Connections:
- net FB_SW: now also U2.5; no longer U2.4
- net NB_SW: now also U2.4; no longer U2.5
Changed lines of the file:
@@
 F 3 "http://www.ti.com/lit/gpn/sn74LS32" H 1500 6900 50  0001 C CNN
 	2    1500 6900
-	1    0    0    -1
+	1    0    0    1
 $EndComp
 Wire Wire Line
