File: HARDWARE/EDA/KICAD/CDJC/_autosave-CDJC.sch (KiCad schematic (older format))
At the start: 55 parts, among them J1 COM_IN, J2 COM_OUT, J3 POWER_IN, J4 POWER_OUT, J5 BIT_OUT, Q1 BC549, SW1 B-SET, U1 74LS04, U2 74LS32, U3 74LS08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

Commit message: U7 pre adjust in PCB
Parts:
- D21: footprint Diode_THT:D_DO-34_SOD68_P7.62mm_Horizontal -> Diode_THT:D_DO-34_SOD68_P12.70mm_Horizontal
Changed lines of the file:
@@
 F 0 "D21" H 8000 4300 50  0000 C CNN
 F 1 "1N4148" H 7550 4300 50  0000 C CNN
-F 2 "Diode_THT:D_DO-34_SOD68_P7.62mm_Horizontal" H 7750 4175 50  0001 C CNN
+F 2 "Diode_THT:D_DO-34_SOD68_P12.70mm_Horizontal" H 7750 4175 50  0001 C CNN
 F 3 "https://assets.nexperia.com/documents/data-sheet/1N4148_1N4448.pdf" H 7750 4350 50  0001 C CNN
 	1    7750 4350
