File: HARDWARE/EDA/KICAD/CDJC/CDJC_Autorouting-test.kicad_pcb (KiCad board)
At the start: 2 copper layers, 91.2 x 100 mm, 55 parts, among them J1 COM_IN, J2 COM_OUT, J3 POWER_IN, J4 POWER_OUT, J5 BIT_OUT, Q1 BC549, SW1 B-SET, U1 74LS04, U2 74LS32, U3 74LS08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

Commit message: PCB finished
Parts:
- moved U1 24.9 mm to (184.6, 98.3), turned to 180 degrees
- moved U3 23.1 mm to (184.6, 69.7), turned to 180 degrees
- moved U4 9.03 mm to (160.6, 69.7), turned to 180 degrees
- moved D2 8.38 mm to (148.1, 135.5)
- moved D3 8.38 mm to (148.1, 130.9)
- moved R1 8.38 mm to (152.8, 138.4)
- moved D1 8.38 mm to (148.1, 140.1)
- moved R2 8.38 mm to (152.8, 133.6)
- moved R3 8.38 mm to (152.8, 128.8)
- moved R4 8.38 mm to (160.4, 140.8)
- moved R5 8.38 mm to (160.4, 136.0)
- moved R6 8.38 mm to (160.4, 131.2)
- moved SW1 8.38 mm to (148.3, 119.5)
- moved U2 3.22 mm to (160.6, 98.3), turned to 180 degrees
- moved D5 2.89 mm to (168.6, 132.3)
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Routing:
- net +5VD: track 368.1 -> 171.4 mm, vias 16 -> 8
- net GNDD: track 443.2 -> 270.2 mm, vias 22 -> 12
- net LB_SW: track 164.6 -> 18.8 mm, vias 6 -> 0
- net LBMon: track 156.2 -> 18.0 mm, vias 4 -> 0
- net ELMon: track 136.6 -> 0.00 mm, vias 4 -> 0
- net FBMon: track 134.1 -> 0.00 mm, vias 8 -> 0
- net Net-(D10-Pad1): track 142.8 -> 21.6 mm, vias 4 -> 0
- net NBMon: track 119.1 -> 0.17 mm, vias 4 -> 0
- net Net-(U4-Pad11): track 103.9 -> 0.00 mm, vias 4 -> 0
- net MRLMon: track 101.0 -> 0.00 mm, vias 2 -> 0
- net FB_SW: track 114.9 -> 15.1 mm
- net NB_SW: track 95.6 -> 17.4 mm, vias 4 -> 0
- net Net-(U1-Pad6): track 55.9 -> 0.00 mm, vias 2 -> 0
- net Net-(U1-Pad2): track 54.4 -> 0.00 mm, vias 4 -> 0
- net Net-(U1-Pad4): track 41.6 -> 0.00 mm, vias 2 -> 0
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Other:
- board size 91.2 x 100 mm -> 100 x 100 mm
